Commit message: added full robot to xacro and works in rviz!

File: turtle_brick/urdf/turtle.urdf.xacro (robot description, xacro)
@@ -1,10 +1,61 @@
 <?xml version="1.0"?>
-<robot xmlns:xacro="http://www.ros.org/wiki/xacro" name="firefighter">
+<robot xmlns:xacro="http://www.ros.org/wiki/xacro" name="turtle">
+  <link name="wheel">
+    <visual>
+      <geometry>
+        <cylinder length="0.1" radius="0.3"/>
+      </geometry>
+      <origin rpy="0 -1.57075 0" xyz="0 0 0.3"/>
+    </visual>
+  </link>
+  <link name="stem">
+    <visual>
+      <geometry>
+        <cylinder length="0.2" radius="0.05"/>
+      </geometry>
+    </visual>
+  </link>
+  <joint name="wheel_to_stem" type="fixed">
+    <parent link="wheel"/>
+    <child link="stem"/>
+    <origin rpy="0 0 0" xyz="0 0 0.7"/>
+  </joint>
   <link name="base_link">
     <visual>
       <geometry>
-        <cylinder length="0.6" radius="0.2"/>
+        <box size="0.4 0.4 0.4"/>
       </geometry>
     </visual>
   </link>
+  <joint name="stem_to_base" type="continuous">
+    <parent link="stem"/>
+    <child link="base_link"/>
+    <axis xyz="0 0 1"/>
+    <origin rpy="0 0 0" xyz="0 0 0.3"/>
+  </joint>
+  <link name="offset">
+    <visual>
+      <geometry>
+        <cylinder length="0.6" radius="0.05"/>
+      </geometry>
+    </visual>
+  </link>
+  <joint name="base_to_offset" type="fixed">
+    <parent link="base_link"/>
+    <child link="offset"/>
+    <origin rpy="0 0 0" xyz="0 0 0.5"/>
+  </joint>
+  <link name="platform">
+    <visual>
+      <geometry>
+        <box size="0.8 0.8 0.05"/>
+      </geometry>
+    </visual>
+  </link>
+  <joint name="offset_to_platform" type="continuous">
+    <parent link="offset"/>
+    <child link="platform"/>
+    <axis xyz="1 1 1"/>
+    <origin rpy="0 0 0" xyz="0 0 0.325"/>
+  </joint>
 </robot>

Commit message: working with new launch file! i uncommented joint_state_publishers and and currently making my own in turtle_robot file

File: turtle_brick/urdf/turtle.urdf.xacro (robot description, xacro)
@@ -1,10 +1,9 @@
 <?xml version="1.0"?>
 <robot xmlns:xacro="http://www.ros.org/wiki/xacro" name="turtle">
-  <link name="wheel">
+  <link name="base_link">
     <visual>
       <geometry>
-        <cylinder length="0.1" radius="0.3"/>
+        <box size="0.4 0.4 0.4"/>
       </geometry>
-      <origin rpy="0 -1.57075 0" xyz="0 0 0.3"/>
     </visual>
   </link>
@@ -16,21 +15,22 @@
     </visual>
   </link>
-  <joint name="wheel_to_stem" type="fixed">
-    <parent link="wheel"/>
+  <joint name="base_to_stem" type="continuous">
+    <parent link="base_link"/>
     <child link="stem"/>
-    <origin rpy="0 0 0" xyz="0 0 0.7"/>
+    <axis xyz="0 0 -1"/>
+    <origin rpy="0 0 0" xyz="0 0 -0.3"/>
   </joint>
-  <link name="base_link">
+  <link name="wheel">
     <visual>
       <geometry>
-        <box size="0.4 0.4 0.4"/>
+        <cylinder length="0.1" radius="0.3"/>
       </geometry>
+      <origin rpy="0 -1.57075 0" xyz="0 0 0.3"/>
     </visual>
   </link>
-  <joint name="stem_to_base" type="continuous">
+  <joint name="stem_to_wheel" type="fixed">
     <parent link="stem"/>
-    <child link="base_link"/>
-    <axis xyz="0 0 1"/>
-    <origin rpy="0 0 0" xyz="0 0 0.3"/>
+    <child link="wheel"/>
+    <origin rpy="0 0 0" xyz="0 0 -0.7"/>
   </joint>
   <link name="offset">

Commit message: I can't spell!!! AHHHHHH fym!!!!!

File: turtle_brick/urdf/turtle.urdf.xacro (robot description, xacro)
@@ -5,4 +5,18 @@
       <geometry>
         <box size="0.4 0.4 0.4"/>
+      </geometry>
+    </visual>
+  </link>
+  <link name="offset">
+    <visual>
+      <geometry>
+        <cylinder length="0.6" radius="0.05"/>
+      </geometry>
+    </visual>
+  </link>
+  <link name="platform">
+    <visual>
+      <geometry>
+        <box size="0.8 0.8 0.05"/>
       </geometry>
     </visual>
@@ -15,10 +29,4 @@
     </visual>
   </link>
-  <joint name="base_to_stem" type="continuous">
-    <parent link="base_link"/>
-    <child link="stem"/>
-    <axis xyz="0 0 -1"/>
-    <origin rpy="0 0 0" xyz="0 0 -0.3"/>
-  </joint>
   <link name="wheel">
     <visual>
@@ -29,33 +37,26 @@
     </visual>
   </link>
-  <joint name="stem_to_wheel" type="fixed">
+  <joint name="base_to_offset" type="fixed">
+    <origin rpy="0 0 0" xyz="0 0 0.5"/>
+    <parent link="base_link"/>
+    <child link="offset"/>
+  </joint>
+  <joint name="offset_to_platform" type="continuous">
+    <axis xyz="1 1 1"/>
+    <origin rpy="0 0 0" xyz="0 0 0.325"/>
+    <parent link="offset"/>
+    <child link="platform"/>
+  </joint>
+  <joint name="base_to_stem" type="continuous">
+    <axis xyz="0 0 -1"/>
+    <origin rpy="0 0 0" xyz="0 0 -0.3"/>
+    <parent link="base_link"/>
+    <child link="stem"/>
+  </joint>
+  <joint name="stem_to_wheel" type="continuous">
+    <axis xyz="0 0 -1"/>
+    <origin xyz="0 0 -0.7"/>
     <parent link="stem"/>
     <child link="wheel"/>
-    <origin rpy="0 0 0" xyz="0 0 -0.7"/>
-  </joint>
-  <link name="offset">
-    <visual>
-      <geometry>
-        <cylinder length="0.6" radius="0.05"/>
-      </geometry>
-    </visual>
-  </link>
-  <joint name="base_to_offset" type="fixed">
-    <parent link="base_link"/>
-    <child link="offset"/>
-    <origin rpy="0 0 0" xyz="0 0 0.5"/>
-  </joint>
-  <link name="platform">
-    <visual>
-      <geometry>
-        <box size="0.8 0.8 0.05"/>
-      </geometry>
-    </visual>
-  </link>
-  <joint name="offset_to_platform" type="continuous">
-    <parent link="offset"/>
-    <child link="platform"/>
-    <axis xyz="1 1 1"/>
-    <origin rpy="0 0 0" xyz="0 0 0.325"/>
   </joint>
 </robot>

Commit message: platform tilts with a message from catcher!

File: turtle_brick/urdf/turtle.urdf.xacro (robot description, xacro)
@@ -43,5 +43,5 @@
   </joint>
   <joint name="offset_to_platform" type="continuous">
-    <axis xyz="1 1 1"/>
+    <axis xyz="1 0 0"/>
     <origin rpy="0 0 0" xyz="0 0 0.325"/>
     <parent link="offset"/>

Commit message: wheel spins!

File: turtle_brick/urdf/turtle.urdf.xacro (robot description, xacro)
@@ -34,5 +34,5 @@
         <cylinder length="0.1" radius="0.3"/>
       </geometry>
-      <origin rpy="0 -1.57075 0" xyz="0 0 0.3"/>
+      <origin rpy="0 -1.57075 0"/>
     </visual>
   </link>
@@ -55,6 +55,6 @@
   </joint>
   <joint name="stem_to_wheel" type="continuous">
-    <axis xyz="0 0 -1"/>
-    <origin xyz="0 0 -0.7"/>
+    <axis xyz="1 0 0"/>
+    <origin xyz="0 0 -0.4"/>
     <parent link="stem"/>
     <child link="wheel"/>

Commit message: yaml works in xacro!!

File: turtle_brick/urdf/turtle.urdf.xacro (robot description, xacro)
@@ -1,4 +1,10 @@
 <?xml version="1.0"?>
 <robot xmlns:xacro="http://www.ros.org/wiki/xacro" name="turtle">
+<xacro:property name="yaml_file" value="$(find turtle_brick)/turtle.yaml" />
+<xacro:property name="props" value="${load_yaml(yaml_file)}" />
+<xacro:property name="start" value="${props['/**']}"/>
+<xacro:property name="ros__parameters" value="${start['ros__parameters']}"/>
+<xacro:property name="platform_height" value="${ros__parameters['platform_height']}"/>
+<xacro:property name="wheel_radius" value="${ros__parameters['wheel_radius']}"/>
   <link name="base_link">
     <visual>
@@ -11,5 +17,5 @@
     <visual>
       <geometry>
-        <cylinder length="0.6" radius="0.05"/>
+        <cylinder length="${platform_height - 0.05 - 0.2  - 0.4 - wheel_radius}" radius="0.05"/>
       </geometry>
     </visual>
@@ -32,5 +38,5 @@
     <visual>
       <geometry>
-        <cylinder length="0.1" radius="0.3"/>
+        <cylinder length="0.1" radius="${wheel_radius}"/>
       </geometry>
       <origin rpy="0 -1.57075 0"/>
